File: Diagrams/blackbox/Microcontroller.kicad_sch (KiCad schematic)
At the start: 2 parts, among them U8 RAZOR 9dof IMU, U9 BNO055

Commit message: Blackbox Diagram V1.1
Parts:
- removed U8: RAZOR 9dof IMU, symbol bitirme:Sparkfun_IMU_Razor
- removed U9: BNO055, symbol bitirme:Sparkfun_IMU_Razor
Connections:
- no-connect marks 0 -> 9
Other:
- note added: "Jetson NANO"
- note added: "POWER SUPPLY"
- note added: "PWM OUTPUT FOR MOTOR DRIVER"
- note added: "USB ARRAY"
