File: Diagrams/blackbox/blackbox.kicad_sch (KiCad schematic)
At the start: 5 parts, among them U1 RAZOR 9dof IMU, U2 BNO055, U3 RPLidar, U4 UBlox M6, U5 Ebyte E22

Commit message: Blackbox Diagram V1 Completed
Top to Down Blok Şeması Oluşturulmuştur. Oluşturulan Hiyerarşik Yapının PDF Çıktısı Oluşturulmuştur.
Parts:
- removed U1: RAZOR 9dof IMU, symbol bitirme:Sparkfun_IMU_Razor
- removed U2: BNO055, symbol bitirme:Sparkfun_IMU_Razor
- removed U3: RPLidar, symbol bitirme:Sparkfun_IMU_Razor
- removed U4: UBlox M6, symbol bitirme:Sparkfun_IMU_Razor
- removed U5: Ebyte E22, symbol bitirme:Sparkfun_IMU_Razor
- added U4: ~, symbol bitirme:USBtoTTL
Connections:
- new net GPS_Base/GND: U4. (VCC)
- new net GPS_Base/V_USB: U4. (VCC)
- new net Microcontroller_Base/USB_2: U4. (VCC)
Other:
- removed sheet Microcontroller
- added sheet Actuator (Actuator.kicad_sch)
- added sheet Base_Lora (base_lora.kicad_sch)
- added sheet GPS_Base (GPS_Base.kicad_sch)
- added sheet LoRa (lora.kicad_sch)
- added sheet Microcontroller_Base (Microcontroller_Base.kicad_sch)
- added sheet Sensors (sensors.kicad_sch)
- added sheet microcontroller (microcontroller.kicad_sch)
- note added: "(Antenna Gain + Power)"
- note added: "Environment"
- note added: "FreeSpace Path Loss (distance)"
- note added: "MotorDriver"
- note added: "Sensors"
- note removed: "IMU'S"
- note removed: "LIDAR"
- title: (none) -> BlackBox Diagram of Autonomous Rover using LoRa Based RTK 

Commit message: Blackbox Diagram V1.1
Connections:
- no-connect marks 0 -> 2
Other:
- sheet Microcontroller_Base renamed SingleBoardComputer_Base
- sheet microcontroller renamed SingleBoardComputer - Rover
- sheet SingleBoardComputer - Rover ports: added USB_4, USB_[1..3]; removed USB_[1..4]
- note added: "BASE"
- note added: "OPTIONAL COMMMUNICATION"
- note added: "ROVER"
- note added: "SBC"
- moved on the sheet: U4
