File: Diagrams/blackbox/lidar.kicad_sch (KiCad schematic)
At the start: 1 part, among them U6 RPLidar

Commit message: Blackbox Diagram V1.1
Other:
- moved on the sheet: U6
Changed lines of the file:
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@@
     (comment 9 "TOLGA")
   )
-  (bus_entry (at 120.65 83.82) (size 2.54 2.54)
+  (bus_entry (at 45.72 95.25) (size 2.54 2.54)
     (stroke (width 0) (type default) (color 0 194 0 1))
   )
-  (bus_entry (at 120.65 81.28) (size 2.54 2.54)
+  (bus_entry (at 45.72 92.71) (size 2.54 2.54)
     (stroke (width 0) (type default) (color 0 0 194 1))
   )
-  (wire (pts (xy 124.46 88.9) (xy 128.27 88.9))
+  (wire (pts (xy 49.53 100.33) (xy 53.34 100.33))
     (stroke (width 0.5) (type default) (color 0 0 0 1))
   )
-  (wire (pts (xy 120.65 49.53) (xy 125.73 49.53))
+  (wire (pts (xy 45.72 60.96) (xy 50.8 60.96))
     (stroke (width 0) (type default))
   )
-  (bus (pts (xy 120.65 81.28) (xy 120.65 83.82))
+  (bus (pts (xy 45.72 92.71) (xy 45.72 95.25))
     (stroke (width 0) (type default))
   )
-  (wire (pts (xy 120.65 54.61) (xy 127 54.61))
+  (wire (pts (xy 45.72 66.04) (xy 52.07 66.04))
     (stroke (width 0) (type default))
   )
-  (wire (pts (xy 123.19 86.36) (xy 128.27 86.36))
+  (wire (pts (xy 48.26 97.79) (xy 53.34 97.79))
     (stroke (width 0) (type default))
   )
-  (wire (pts (xy 124.46 78.74) (xy 124.46 81.28))
+  (wire (pts (xy 49.53 90.17) (xy 49.53 92.71))
     (stroke (width 0.5) (type default) (color 132 0 0 1))
   )
-  (wire (pts (xy 124.46 81.28) (xy 128.27 81.28))
+  (wire (pts (xy 49.53 92.71) (xy 53.34 92.71))
     (stroke (width 0.5) (type default) (color 132 0 0 1))
   )
-  (bus (pts (xy 120.65 80.01) (xy 120.65 81.28))
+  (bus (pts (xy 45.72 91.44) (xy 45.72 92.71))
     (stroke (width 0) (type default))
   )
-  (wire (pts (xy 124.46 88.9) (xy 124.46 90.17))
+  (wire (pts (xy 49.53 100.33) (xy 49.53 101.6))
     (stroke (width 0.5) (type default) (color 0 0 0 1))
   )
-  (wire (pts (xy 123.19 83.82) (xy 128.27 83.82))
+  (wire (pts (xy 48.26 95.25) (xy 53.34 95.25))
     (stroke (width 0) (type default) (color 0 0 194 1))
   )
-  (rectangle (start 109.22 63.5) (end 173.99 104.14)
+  (rectangle (start 34.29 74.93) (end 99.06 115.57)
     (stroke (width 0) (type default))
     (fill (type none))
   )
-  (image (at 147.32 85.09) (scale 0.451172)
+  (image (at 72.39 96.52) (scale 0.451172)
     (data
       iVBORw0KGgoAAAANSUhEUgAAAZAAAAGQCAIAAAAP3aGbAAAAA3NCSVQICAjb4U/gAAAACXBIWXMA
@@
     )
   )
-  (hierarchical_label "UART-1" (shape input) (at 120.65 80.01 180) (fields_autoplaced)
+  (hierarchical_label "UART-1" (shape input) (at 45.72 91.44 180) (fields_autoplaced)
     (effects (font (size 1.27 1.27)) (justify right))
   )
-  (hierarchical_label "GND" (shape input) (at 120.65 54.61 180) (fields_autoplaced)
+  (hierarchical_label "GND" (shape input) (at 45.72 66.04 180) (fields_autoplaced)
     (effects (font (size 1.27 1.27)) (justify right))
   )
-  (hierarchical_label "V_USB" (shape input) (at 120.65 49.53 180) (fields_autoplaced)
+  (hierarchical_label "V_USB" (shape input) (at 45.72 60.96 180) (fields_autoplaced)
     (effects (font (size 1.27 1.27)) (justify right))
   )
-  (symbol (lib_id "power:VBUS") (at 125.73 49.53 270) (unit 1)
+  (symbol (lib_id "power:VBUS") (at 50.8 60.96 270) (unit 1)
     (in_bom yes) (on_board yes) (dnp no) (fields_autoplaced)
-    (property "Reference" "#PWR013" (at 121.92 49.53 0)
-      (effects (font (size 1.27 1.27)) hide)
-    )
-    (property "Value" "VBUS" (at 129.54 49.53 90)
+    (property "Reference" "#PWR013" (at 46.99 60.96 0)
+      (effects (font (size 1.27 1.27)) hide)
+    )
+    (property "Value" "VBUS" (at 54.61 60.96 90)
       (effects (font (size 1.27 1.27)) (justify left))
     )
-    (property "Footprint" "" (at 125.73 49.53 0)
-      (effects (font (size 1.27 1.27)) hide)
-    )
-    (property "Datasheet" "" (at 125.73 49.53 0)
+    (property "Footprint" "" (at 50.8 60.96 0)
+      (effects (font (size 1.27 1.27)) hide)
+    )
+    (property "Datasheet" "" (at 50.8 60.96 0)
       (effects (font (size 1.27 1.27)) hide)
     )
@@
     )
   )
-  (symbol (lib_id "power:GND") (at 127 54.61 90) (unit 1)
+  (symbol (lib_id "power:GND") (at 52.07 66.04 90) (unit 1)
     (in_bom yes) (on_board yes) (dnp no)
-    (property "Reference" "#PWR014" (at 133.35 54.61 0)
-      (effects (font (size 1.27 1.27)) hide)
-    )
-    (property "Value" "GND" (at 130.81 54.61 0)
+    (property "Reference" "#PWR014" (at 58.42 66.04 0)
+      (effects (font (size 1.27 1.27)) hide)
+    )
+    (property "Value" "GND" (at 55.88 66.04 0)
       (effects (font (size 1.27 1.27)))
     )
-    (property "Footprint" "" (at 127 54.61 0)
-      (effects (font (size 1.27 1.27)) hide)
-    )
-    (property "Datasheet" "" (at 127 54.61 0)
+    (property "Footprint" "" (at 52.07 66.04 0)
+      (effects (font (size 1.27 1.27)) hide)
+    )
+    (property "Datasheet" "" (at 52.07 66.04 0)
       (effects (font (size 1.27 1.27)) hide)
     )
@@
     )
   )
-  (symbol (lib_id "power:VBUS") (at 124.46 78.74 0) (unit 1)
+  (symbol (lib_id "power:VBUS") (at 49.53 90.17 0) (unit 1)
     (in_bom yes) (on_board yes) (dnp no) (fields_autoplaced)
-    (property "Reference" "#PWR011" (at 124.46 82.55 0)
-      (effects (font (size 1.27 1.27)) hide)
-    )
-    (property "Value" "VBUS" (at 124.46 73.66 0)
+    (property "Reference" "#PWR011" (at 49.53 93.98 0)
+      (effects (font (size 1.27 1.27)) hide)
+    )
+    (property "Value" "VBUS" (at 49.53 85.09 0)
       (effects (font (size 1.27 1.27)))
     )
-    (property "Footprint" "" (at 124.46 78.74 0)
-      (effects (font (size 1.27 1.27)) hide)
-    )
-    (property "Datasheet" "" (at 124.46 78.74 0)
+    (property "Footprint" "" (at 49.53 90.17 0)
+      (effects (font (size 1.27 1.27)) hide)
+    )
+    (property "Datasheet" "" (at 49.53 90.17 0)
       (effects (font (size 1.27 1.27)) hide)
     )
@@
     )
   )
-  (symbol (lib_id "power:GND") (at 124.46 90.17 0) (unit 1)
+  (symbol (lib_id "power:GND") (at 49.53 101.6 0) (unit 1)
     (in_bom yes) (on_board yes) (dnp no)
-    (property "Reference" "#PWR012" (at 124.46 96.52 0)
-      (effects (font (size 1.27 1.27)) hide)
-    )
-    (property "Value" "GND" (at 124.46 93.98 0)
+    (property "Reference" "#PWR012" (at 49.53 107.95 0)
+      (effects (font (size 1.27 1.27)) hide)
+    )
+    (property "Value" "GND" (at 49.53 105.41 0)
       (effects (font (size 1.27 1.27)))
     )
-    (property "Footprint" "" (at 124.46 90.17 0)
-      (effects (font (size 1.27 1.27)) hide)
-    )
-    (property "Datasheet" "" (at 124.46 90.17 0)
+    (property "Footprint" "" (at 49.53 101.6 0)
+      (effects (font (size 1.27 1.27)) hide)
+    )
+    (property "Datasheet" "" (at 49.53 101.6 0)
       (effects (font (size 1.27 1.27)) hide)
     )
@@
     )
   )
-  (symbol (lib_name "Sparkfun_IMU_Razor_2") (lib_id "bitirme:Sparkfun_IMU_Razor") (at 129.54 77.47 0) (unit 1)
+  (symbol (lib_name "Sparkfun_IMU_Razor_2") (lib_id "bitirme:Sparkfun_IMU_Razor") (at 54.61 88.9 0) (unit 1)
     (in_bom yes) (on_board yes) (dnp no)
-    (property "Reference" "U6" (at 133.35 76.2 0)
+    (property "Reference" "U6" (at 58.42 87.63 0)
       (effects (font (size 1.27 1.27)) (justify left))
     )
-    (property "Value" "RPLidar" (at 166.37 85.09 0)
+    (property "Value" "RPLidar" (at 91.44 96.52 0)
       (effects (font (size 1.27 1.27)))
     )
-    (property "Footprint" "" (at 129.54 77.47 0)
-      (effects (font (size 1.27 1.27)) hide)
-    )
-    (property "Datasheet" "https://cdn.sparkfun.com/assets/e/a/f/9/8/LD208_SLAMTEC_rplidar_datasheet_A2M8_v1.0_en.pdf" (at 129.54 77.47 0)
-      (effects (font (size 1.27 1.27)) hide)
-    )
-    (property "Website" "https://market.samm.com/sparkfun-rplidar-a2m8-360-lazer-mesafe-tarayici" (at 129.54 77.47 0)
-      (effects (font (size 1.27 1.27)) hide)
-    )
+    (property "Footprint" "" (at 54.61 88.9 0)
+      (effects (font (size 1.27 1.27)) hide)
+    )
+    (property "Datasheet" "https://cdn.sparkfun.com/assets/e/a/f/9/8/LD208_SLAMTEC_rplidar_datasheet_A2M8_v1.0_en.pdf" (at 54.61 88.9 0)
+      (effects (font (size 1.27 1.27)) hide)
+    )
+    (property "Website" "https://market.samm.com/sparkfun-rplidar-a2m8-360-lazer-mesafe-tarayici" (at 54.61 88.9 0)
+      (effects (font (size 1.27 1.27)) hide)
+    )
