Commit message: feat: with obstacle avoindece

File: src/kuzu_robot/urdf/kuzu_robot.urdf (robot description, URDF)
Before this commit: robot kuzu_robot, 6 links, 5 joints
Links:
- removed link front_left_wheel
- removed link front_right_wheel
- removed link rear_left_wheel
- removed link rear_right_wheel
Joints:
- removed joint rear_left_wheel_joint
- removed joint rear_right_wheel_joint
- removed joint steering_fl_joint
- removed joint steering_fr_joint
